Commit message: URDF working

File: ros_ws/src/urdf_project/urdf/urdf_project.urdf (robot description, URDF)
Before this commit: robot urdf_project, 4 links, 3 joints
Links:
- added link link_0; collision cylinder length=10 radius=0.5; visual cylinder length=10 radius=0.5
- link link_1: geometry collision cylinder length=10 radius=0.5; visual cylinder length=10 radius=0.5
- link link_2: geometry collision box size=2.5 2.5 2.5; visual box size=2.5 2.5 2.5
Joints:
- added joint base_joint: type fixed, parent world, child base_link, origin xyz=0 0 1.0 rpy=0 0 0
- joint J0: child base_link -> link_0; parent world -> base_link
- joint J1: axis 0 0 1 -> 0 1 0; limit lower=0.0 upper=6.2831853 effort=0.0 velocity=0.0 -> lower=-0.7853981625 upper=3.9269908125 effort=0.0 velocity=0.0; origin xyz=0.0 0.0 0.0 rpy=-1.5708 0 0 -> xyz=0.0 0.0 10.0 rpy=0 -1.5708 0; parent base_link -> link_0
- joint J2: origin xyz=0.0 0.0 0.0 rpy=0 1.5708 0 -> xyz=0.0 0.0 10.0 rpy=0 0 0

Commit message: Screenshots, adjusted robot size

File: ros_ws/src/urdf_project/urdf/urdf_project.urdf (robot description, URDF)
Before this commit: robot urdf_project, 5 links, 4 joints
Links:
- link link_0: geometry collision cylinder length=3.0 radius=0.5; visual cylinder length=3.0 radius=0.5
- link link_1: geometry collision cylinder length=3.0 radius=0.5; visual cylinder length=3.0 radius=0.5
- link link_2: geometry collision box size=1.0 1.0 1.0; visual box size=1.0 1.0 1.0
Joints:
- joint J1: origin xyz=0.0 0.0 10.0 rpy=0 -1.5708 0 -> xyz=0.0 0.0 3.0 rpy=0 -1.5708 0
- joint J2: origin xyz=0.0 0.0 10.0 rpy=0 0 0 -> xyz=0.0 0.0 3.0 rpy=0 0 0
